File: T41_V012_Files_01-15-24/T41_V012_KiCad/T41-main-board-V012/T41-main-board-V012.kicad_pcb (KiCad board)
At the start: 4 copper layers, 100 x 100 mm, 103 parts, among them J1 +12V, J10 Conn_01x02, J11 ENCODER, J12 BANDS, J13 Header, J14 Rec_Out, J15 Rec_In, J16 Mic_In, J17 Ex_Out, J18 Conn_01x02, J19 Conn_01x01, J2 Fan1, J20 Conn_01x01, J21 Conn_01x01, J22 Header, J23 Ethernet, J24 USBHost, J3 Acc, J4 12-13.8V, J5 Front Panel, J6 RF CONTROL, J7 Display, J8 Display Voltage, J9 Keys/PTT, Q1 IRF4905, Q2 2N7000, Q3 2N7000, SW1 ON-OFF BUTTON, U1 LM7805CT, U10 LM1117T-3.3, U2 AP7384-50V, U3 LM1117T-3.3, U4 ATtiny85-20S, U5 PCM5102, U6 PCM1808PW, U8 Teensy4.1, U9 LM7805CT

Commit message: Moved voltage regulator on main board so no interference with Teensy audio hat
Parts:
- moved C2 20.7 mm to (99.9, 135.4), turned to 180 degrees
- moved J8 17.3 mm to (99.6, 126.2)
- moved D2 15.9 mm to (93.3, 116.8)
- moved R8 15.9 mm to (93.3, 119.6)
- moved C1 14.6 mm to (96.9, 139.7)
- moved D3 12.0 mm to (99.9, 129.8)
- moved H1 12.0 mm to (110.6, 120.4)
- moved H2 12.0 mm to (110.6, 145.8)
- moved R9 12.0 mm to (100.0, 132.3)
- moved U1 12.0 mm to (114.0, 135.6)
- moved U9 12.0 mm to (107.2, 135.6)
Routing:
- net Net-(J7-Pin_7): track 84.7 -> 103.1 mm
- net +5V: track 150.1 -> 132.4 mm
- net +3V3: track 263.5 -> 280.6 mm
- net +12V: track 167.3 -> 162.5 mm
- net Net-(U1-VO): track 47.6 -> 49.4 mm
- net GND: vias 139 -> 142
Other:
- board text added: "T41 Main+, V012.6 Design by AC8GY/W8TEE/K9HZ KiCad Layout by KI3P 4 layer, 2024-01-26"
- board text added: "TX"
- board text removed: "T41 Main+, V012.6 Design by AC8GY/W8TEE/K9HZ KiCad Layout by KI3P 4 layer, 2024-01-14"
